File: Adapter-Pfostenstecker.kicad_pcb (KiCad board)
At the start: 2 copper layers, 12.7 x 22.9 mm, 3 parts, among them J1001 Conn_02x08_Odd_Even, J1002 Conn_01x08, J1003 Conn_01x08

Commit message: update
Parts:
- moved J1001 131.5 mm to (26.0, 20.2)
- moved J1002 131.5 mm to (31.1, 20.2)
- moved J1003 131.5 mm to (23.5, 20.2)
Changed lines of the file:
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@@
   (net 16 "Net-(J1001-Pin_7)")
   (footprint "Connector_PinHeader_2.54mm:PinHeader_2x08_P2.54mm_Vertical" (layer "F.Cu")
-    (at 147.32 71.12)
+    (at 26.035 20.193)
     (descr "Through hole straight pin header, 2x08, 2.54mm pitch, double rows")
     (tags "Through hole pin header THT 2x08 2.54mm double row")
@@
   )
   (footprint "Connector_PinHeader_2.54mm:PinHeader_1x08_P2.54mm_Vertical" (layer "B.Cu")
-    (at 152.4 71.135 180)
+    (at 31.115 20.208 180)
     (descr "Through hole straight pin header, 1x08, 2.54mm pitch, single row")
     (tags "Through hole pin header THT 1x08 2.54mm single row")
@@
   )
   (footprint "Connector_PinHeader_2.54mm:PinHeader_1x08_P2.54mm_Vertical" (layer "B.Cu")
-    (at 144.78 71.12 180)
+    (at 23.495 20.193 180)
     (descr "Through hole straight pin header, 1x08, 2.54mm pitch, single row")
     (tags "Through hole pin header THT 1x08 2.54mm single row")
@@
     )
   )
-  (gr_line (start 154.94 92.075) (end 142.24 92.075)
-    (stroke (width 0.1) (type default)) (layer "Edge.Cuts"))
-  (gr_line (start 142.24 69.215) (end 154.94 69.215)
-    (stroke (width 0.1) (type default)) (layer "Edge.Cuts"))
-  (gr_line (start 142.24 92.075) (end 142.24 69.215)
-    (stroke (width 0.1) (type default)) (layer "Edge.Cuts"))
-  (gr_line (start 154.94 69.215) (end 154.94 92.075)
-    (stroke (width 0.1) (type default)) (layer "Edge.Cuts"))
-  (gr_text "v1.0\n" (at 148.59 91.059) (layer "B.SilkS")
+  (gr_line (start 33.655 41.148) (end 20.955 41.148)
+    (stroke (width 0.1) (type default)) (layer "Edge.Cuts"))
+  (gr_line (start 20.955 18.288) (end 33.655 18.288)
+    (stroke (width 0.1) (type default)) (layer "Edge.Cuts"))
+  (gr_line (start 20.955 41.148) (end 20.955 18.288)
+    (stroke (width 0.1) (type default)) (layer "Edge.Cuts"))
+  (gr_line (start 33.655 18.288) (end 33.655 41.148)
+    (stroke (width 0.1) (type default)) (layer "Edge.Cuts"))
+  (gr_text "v1.0\n" (at 27.305 40.132) (layer "B.SilkS")
     (effects (font (size 1 1) (thickness 0.25)) (justify mirror))
   )
@@
     (effects (font (size 1.5 1.5) (thickness 0.3)) (justify mirror))
   )
-  (gr_text "©H3-H5N6 '23\n" (at 148.59 91.186) (layer "F.SilkS")
+  (gr_text "©H3-H5N6 '23\n" (at 27.305 40.259) (layer "F.SilkS")
     (effects (font (size 1 1) (thickness 0.25)))
   )
   (dimension (type aligned) (layer "F.CrtYd")
-    (pts (xy 144.78 89.916) (xy 152.4 89.916))
+    (pts (xy 23.495 38.989) (xy 31.115 38.989))
     (height 7.62)
-    (gr_text "7,62 mm" (at 148.59 96.386) (layer "F.CrtYd")
+    (gr_text "7,62 mm" (at 27.305 45.459) (layer "F.CrtYd")
       (effects (font (size 1 1) (thickness 0.15)))
     )
@@
   )
   (dimension (type aligned) (layer "F.CrtYd")
-    (pts (xy 147.32 89.535) (xy 149.86 89.535))
+    (pts (xy 26.035 38.608) (xy 28.575 38.608))
     (height 5.08)
-    (gr_text "2,54 mm" (at 148.59 93.465) (layer "F.CrtYd")
+    (gr_text "2,54 mm" (at 27.305 42.538) (layer "F.CrtYd")
       (effects (font (size 1 1) (thickness 0.15)))
     )
@@
     (style (thickness 0.05) (arrow_length 1.27) (text_position_mode 0) (extension_height 0.58642) (extension_offset 0.5) keep_text_aligned)
   )
-  (segment (start 144.78 71.12) (end 147.32 71.12) (width 1) (layer "B.Cu") (net 1))
-  (segment (start 149.86 71.12) (end 152.4 71.12) (width 1) (layer "B.Cu") (net 2))
-  (segment (start 144.78 73.66) (end 147.32 73.66) (width 1) (layer "B.Cu") (net 3))
-  (segment (start 149.86 73.66) (end 152.4 73.66) (width 1) (layer "B.Cu") (net 4))
-  (segment (start 144.78 76.2) (end 147.32 76.2) (width 1) (layer "B.Cu") (net 5))
-  (segment (start 149.86 76.2) (end 152.4 76.2) (width 1) (layer "B.Cu") (net 6))
-  (segment (start 149.86 78.74) (end 152.4 78.74) (width 1) (layer "B.Cu") (net 7))
-  (segment (start 144.78 81.28) (end 147.32 81.28) (width 1) (layer "B.Cu") (net 8))
-  (segment (start 149.86 81.28) (end 152.4 81.28) (width 1) (layer "B.Cu") (net 9))
-  (segment (start 144.78 83.82) (end 147.32 83.82) (width 1) (layer "B.Cu") (net 10))
-  (segment (start 149.86 83.82) (end 152.4 83.82) (width 1) (layer "B.Cu") (net 11))
-  (segment (start 144.78 86.36) (end 147.32 86.36) (width 1) (layer "B.Cu") (net 12))
-  (segment (start 149.86 88.9) (end 152.4 88.9) (width 1) (layer "B.Cu") (net 13))
-  (segment (start 144.78 88.9) (end 147.32 88.9) (width 1) (layer "B.Cu") (net 14))
-  (segment (start 149.86 86.36) (end 152.4 86.36) (width 1) (layer "B.Cu") (net 15))
-  (segment (start 144.78 78.74) (end 147.32 78.74) (width 1) (layer "B.Cu") (net 16))
+  (segment (start 23.495 20.193) (end 26.035 20.193) (width 1) (layer "B.Cu") (net 1))
+  (segment (start 28.575 20.193) (end 31.115 20.193) (width 1) (layer "B.Cu") (net 2))
+  (segment (start 23.495 22.733) (end 26.035 22.733) (width 1) (layer "B.Cu") (net 3))
+  (segment (start 28.575 22.733) (end 31.115 22.733) (width 1) (layer "B.Cu") (net 4))
+  (segment (start 23.495 25.273) (end 26.035 25.273) (width 1) (layer "B.Cu") (net 5))
+  (segment (start 28.575 25.273) (end 31.115 25.273) (width 1) (layer "B.Cu") (net 6))
+  (segment (start 28.575 27.813) (end 31.115 27.813) (width 1) (layer "B.Cu") (net 7))
+  (segment (start 23.495 30.353) (end 26.035 30.353) (width 1) (layer "B.Cu") (net 8))
+  (segment (start 28.575 30.353) (end 31.115 30.353) (width 1) (layer "B.Cu") (net 9))
+  (segment (start 23.495 32.893) (end 26.035 32.893) (width 1) (layer "B.Cu") (net 10))
+  (segment (start 28.575 32.893) (end 31.115 32.893) (width 1) (layer "B.Cu") (net 11))
+  (segment (start 23.495 35.433) (end 26.035 35.433) (width 1) (layer "B.Cu") (net 12))
+  (segment (start 28.575 37.973) (end 31.115 37.973) (width 1) (layer "B.Cu") (net 13))
+  (segment (start 23.495 37.973) (end 26.035 37.973) (width 1) (layer "B.Cu") (net 14))
+  (segment (start 28.575 35.433) (end 31.115 35.433) (width 1) (layer "B.Cu") (net 15))
+  (segment (start 23.495 27.813) (end 26.035 27.813) (width 1) (layer "B.Cu") (net 16))
 )
